Commit message: exercise 1.1

File: urdf/reemc_full_ft_hey5.urdf (robot description, URDF)
Before this commit: robot reemc, 132 links, 131 joints
Links:
- link arm_left_2_link: geometry collision mesh filename=package://reemc_description/meshes/arm/arm_2_collision.stl scale=1 2 1.0; visual mesh filename=package://reemc_description/meshes/arm/arm_2.dae scale=1 2 1.0
- link arm_left_3_link: geometry collision mesh filename=package://reemc_description/meshes/arm/arm_3_collision.stl scale=1 1 2.0; visual mesh filename=package://reemc_description/meshes/arm/arm_3.dae scale=1 1 2.0
- link arm_left_4_link: geometry collision mesh filename=package://reemc_description/meshes/arm/arm_4_collision.stl scale=2 1 1.0; visual mesh filename=package://reemc_description/meshes/arm/arm_4.dae scale=2 1 1.0
- link arm_left_5_link: geometry collision mesh filename=package://reemc_description/meshes/arm/arm_5_collision.stl scale=1 1 2.0; visual mesh filename=package://reemc_description/meshes/arm/arm_5.dae scale=1 1 2.0
- link arm_left_6_link: geometry collision cylinder length=0.0385 radius=0.04; visual mesh filename=package://reemc_description/meshes/arm/arm_6.dae scale=1 2 1.0
Joints:
- joint arm_left_3_joint: origin xyz=0.02 -0.142 0 rpy=-1.57079632679 0 0 -> xyz=0.02 -0.3 0 rpy=-1.57079632679 0 0
- joint arm_left_4_joint: origin xyz=0 -0.02 -0.088 rpy=0 -1.57079632679 0 -> xyz=0 -0.02 -0.17 rpy=0 -1.57079632679 0
- joint arm_left_5_joint: origin xyz=-0.088 0.02 0 rpy=0 1.57079632679 0 -> xyz=-0.17 0.02 0 rpy=0 1.57079632679 0
- joint arm_left_6_joint: origin xyz=0 0 -0.15 rpy=1.57079632679 0 0 -> xyz=0 0 -0.3 rpy=1.57079632679 0 0

Commit message: undoes old urdf changes

File: urdf/reemc_full_ft_hey5.urdf (robot description, URDF)
Before this commit: robot reemc, 132 links, 131 joints
Links:
- link arm_left_2_link: geometry collision mesh filename=package://reemc_description/meshes/arm/arm_2_collision.stl scale=1 1 1.0; visual mesh filename=package://reemc_description/meshes/arm/arm_2.dae scale=1 1 1.0
- link arm_left_3_link: geometry collision mesh filename=package://reemc_description/meshes/arm/arm_3_collision.stl scale=1 1 1.0; visual mesh filename=package://reemc_description/meshes/arm/arm_3.dae scale=1 1 1.0
- link arm_left_4_link: geometry collision mesh filename=package://reemc_description/meshes/arm/arm_4_collision.stl scale=1 1 1.0; visual mesh filename=package://reemc_description/meshes/arm/arm_4.dae scale=1 1 1.0
- link arm_left_5_link: geometry collision mesh filename=package://reemc_description/meshes/arm/arm_5_collision.stl scale=1 1 1.0; visual mesh filename=package://reemc_description/meshes/arm/arm_5.dae scale=1 1 1.0
- link arm_left_6_link: geometry collision cylinder length=0.0385 radius=0.04; visual mesh filename=package://reemc_description/meshes/arm/arm_6.dae scale=1 1 1.0
Joints:
- joint arm_left_3_joint: origin xyz=0.02 -0.3 0 rpy=-1.57079632679 0 0 -> xyz=0.02 -0.142 0 rpy=-1.57079632679 0 0
- joint arm_left_4_joint: origin xyz=0 -0.02 -0.17 rpy=0 -1.57079632679 0 -> xyz=0 -0.02 -0.088 rpy=0 -1.57079632679 0
- joint arm_left_5_joint: origin xyz=-0.17 0.02 0 rpy=0 1.57079632679 0 -> xyz=-0.088 0.02 0 rpy=0 1.57079632679 0
- joint arm_left_6_joint: origin xyz=0 0 -0.3 rpy=1.57079632679 0 0 -> xyz=0 0 -0.15 rpy=1.57079632679 0 0
